File: Kicad/Sub_UC.kicad_sch (KiCad schematic)
At the start: 43 parts, among them J12 Screw_Terminal_01x02, J13 Screw_Terminal_01x02, J14 Screw_Terminal_01x02, J15 Screw_Terminal_01x02, J17 Screw_Terminal_01x02, J18 Screw_Terminal_01x02, J19 Screw_Terminal_01x02, J20 Screw_Terminal_01x02, Q1 BC547, Q2 BC547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

Commit message: Correction demodulateur TIC
Parts:
- R103: value 100k -> 4k7
- R76: value 4k7 -> 1k
Changed lines of the file:
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@@
 			)
 		)
-		(property "Value" "100k"
+		(property "Value" "4k7"
 			(at 211.074 143.51 0)
 			(effects
@@
 			)
 		)
-		(property "Value" "4k7"
+		(property "Value" "1k"
 			(at 238.76 131.064 90)
 			(effects
